File: pcb/eth_shield_W5100/eth_shield_W5100.sch (KiCad schematic (older format))
At the start: 46 parts, among them J1 Conn_02x05_Odd_Even, J2 HR911105A, U1 LM1117-3.3, U2 W5100, Y1 Crystal

Commit message: Se agraga la asociación de componentes y la netlist
Parts:
- C1: footprint (none) -> Capacitor_SMD:C_0805_2012Metric_Pad1.15x1.40mm_HandSolder
- C10, C11, C12, C13, C14, C15, C16, C17, C18, C2, C3, C4, C5, C6, C7, C8, C9: footprint (none) -> Capacitor_SMD:C_0603_1608Metric_Pad1.05x0.95mm_HandSolder
- D1, D2, D3, D4, D5, D6: footprint (none) -> LED_SMD:LED_0603_1608Metric_Pad1.05x0.95mm_HandSolder
- J1: footprint (none) -> Connector_PinSocket_2.54mm:PinSocket_2x05_P2.54mm_Vertical
- R1, R10, R11, R12, R13, R14, R15, R16, R17, R2, R3, R4, R5, R6, R7, R8, R9: footprint (none) -> Resistor_SMD:R_0603_1608Metric_Pad0.98x0.95mm_HandSolder
- U1: footprint (none) -> Package_TO_SOT_SMD:SOT-223-3_TabPin2
- Y1: footprint (none) -> Crystal:Crystal_HC18-U_Vertical

Commit message: Se termina el routeo, se agregan comentarios y detalles
Parts:
- added FID1, FID2, FID3: Fiducial, Fiducial:Fiducial_0.75mm_Mask1.5mm, symbol Mechanical:Fiducial
- J2: footprint HANRUN_HR911105A -> (none)
Changed lines of the file:
@@
 F 0 "J2" H 10539 2696 50  0000 L CNN
 F 1 "HR911105A" H 10539 2605 50  0000 L CNN
-F 2 "HANRUN_HR911105A" H 9150 2650 50  0001 L BNN
+F 2 "" H 9150 2650 50  0001 L BNN
 F 3 "" H 9150 2650 50  0001 L BNN
 F 4 "HR911105A" H 9150 2650 50  0001 L BNN "MP"
@@
 	2750 3200 2750 3350
 Connection ~ 2750 3350
+$Comp
+L Mechanical:Fiducial FID3
+U 1 1 61131BF2
+P 3500 5700
+F 0 "FID3" H 3585 5746 50  0000 L CNN
+F 1 "Fiducial" H 3585 5655 50  0000 L CNN
+F 2 "Fiducial:Fiducial_0.75mm_Mask1.5mm" H 3500 5700 50  0001 C CNN
+F 3 "~" H 3500 5700 50  0001 C CNN
+	1    3500 5700
+	1    0    0    -1
+$EndComp
+$Comp
+L Mechanical:Fiducial FID2
+U 1 1 611343BC
+P 3500 5450
+F 0 "FID2" H 3585 5496 50  0000 L CNN
+F 1 "Fiducial" H 3585 5405 50  0000 L CNN
+F 2 "Fiducial:Fiducial_0.75mm_Mask1.5mm" H 3500 5450 50  0001 C CNN
+F 3 "~" H 3500 5450 50  0001 C CNN
+	1    3500 5450
+	1    0    0    -1
+$EndComp
+$Comp
+L Mechanical:Fiducial FID1
+U 1 1 611346BF
+P 3500 5200
+F 0 "FID1" H 3585 5246 50  0000 L CNN
+F 1 "Fiducial" H 3585 5155 50  0000 L CNN
+F 2 "Fiducial:Fiducial_0.75mm_Mask1.5mm" H 3500 5200 50  0001 C CNN
+F 3 "~" H 3500 5200 50  0001 C CNN
+	1    3500 5200
+	1    0    0    -1
+$EndComp
 $EndSCHEMATC

Commit message: Se agrega agujeros y se hacen las correciones indicadas por el docente
Parts:
- added H1, H2: MountingHole, MountingHole:MountingHole_2.1mm, symbol Mechanical:MountingHole
Changed lines of the file:
@@
+	1    0    0    -1
+$EndComp
+$Comp
+L Mechanical:MountingHole H2
+U 1 1 6116774E
+P 3500 4900
+F 0 "H2" H 3600 4946 50  0000 L CNN
+F 1 "MountingHole" H 3600 4855 50  0000 L CNN
+F 2 "MountingHole:MountingHole_2.1mm" H 3500 4900 50  0001 C CNN
+F 3 "~" H 3500 4900 50  0001 C CNN
+	1    3500 4900
+	1    0    0    -1
+$EndComp
+$Comp
+L Mechanical:MountingHole H1
+U 1 1 61167DEA
+P 3500 4600
+F 0 "H1" H 3600 4646 50  0000 L CNN
+F 1 "MountingHole" H 3600 4555 50  0000 L CNN
+F 2 "MountingHole:MountingHole_2.1mm" H 3500 4600 50  0001 C CNN
+F 3 "~" H 3500 4600 50  0001 C CNN
+	1    3500 4600
 	1    0    0    -1
 $EndComp

Commit message: Se agregan las correciones que se hicieron para la presentación
Parts:
- J2: symbol HR911105A:HR911105A -> eth_shield_W5100-rescue:HR911105A-HR911105A; Manufacturer (none) -> Phoenix Contact; Manufacturer PN (none) -> 1091946
- U1: Manufacturer (none) -> Texas Instruments; Manufacturer PN (none) -> LM1117IMPX-3.3/NOPB
- U2: Manufacturer (none) -> WIZnet; Manufacturer PN (none) -> W5100
- Y1: Manufacturer (none) -> ECS; Manufacturer PN (none) -> ECS-200-18-4X-CKM
Changed lines of the file:
@@
 encoding utf-8
 Sheet 1 1
-Title "Ethernet W5100"
+Title "Réplica Ethernet W5100"
 Date "2021-07-25"
 Rev "0"
 Comp "Joaquín Ulloa - CESE, FIUBA"
-Comment1 ""
+Comment1 "Revisor: Diego Brengi"
 Comment2 ""
 Comment3 ""
@@
 U 1 1 60F4C459
 P 4900 3400
-F 0 "U2" H 4900 1311 50  0000 C CNN
-F 1 "W5100" H 4900 1220 50  0000 C CNN
+F 0 "U2" H 5200 1450 50  0000 C CNN
+F 1 "W5100" H 4550 1450 50  0000 C CNN
 F 2 "Package_QFP:LQFP-80_10x10mm_P0.4mm" H 5050 1450 50  0001 L CNN
 F 3 "http://www.wiznet.io/wp-content/uploads/wiznethome/Chip/W5100/Document/W5100_Datasheet_v1.2.7.pdf" H 1250 6550 50  0001 C CNN
+F 4 "WIZnet" H 4900 3400 50  0001 C CNN "Manufacturer"
+F 5 "W5100" H 4900 3400 50  0001 C CNN "Manufacturer PN"
 	1    4900 3400
 	1    0    0    -1
@@
 $EndComp
 $Comp
-L HR911105A:HR911105A J2
+L eth_shield_W5100-rescue:HR911105A-HR911105A J2
 U 1 1 60FFE069
 P 9150 2650
@@
 F 10 "Manufacturer Recommendation" H 9150 2650 50  0001 L BNN "STANDARD"
 F 11 "A" H 9150 2650 50  0001 L BNN "PARTREV"
+F 12 "Phoenix Contact" H 9150 2650 50  0001 C CNN "Manufacturer"
+F 13 "1091946" H 9150 2650 50  0001 C CNN "Manufacturer PN"
 	1    9150 2650
 	1    0    0    -1
@@
 U 1 1 61037DCD
 P 6450 2600
-F 0 "R5" H 6520 2646 50  0000 L CNN
-F 1 "49R9" H 6520 2555 50  0000 L CNN
+F 0 "R5" H 6500 2650 50  0000 L CNN
+F 1 "49R9" H 6500 2550 50  0000 L CNN
 F 2 "Resistor_SMD:R_0603_1608Metric_Pad0.98x0.95mm_HandSolder" V 6380 2600 50  0001 C CNN
 F 3 "~" H 6450 2600 50  0001 C CNN
@@
 U 1 1 6103929D
 P 7050 1150
-F 0 "R7" H 6980 1104 50  0000 R CNN
-F 1 "49R9" H 6980 1195 50  0000 R CNN
+F 0 "R7" H 7000 1100 50  0000 R CNN
+F 1 "49R9" H 7000 1200 50  0000 R CNN
 F 2 "Resistor_SMD:R_0603_1608Metric_Pad0.98x0.95mm_HandSolder" V 6980 1150 50  0001 C CNN
 F 3 "~" H 7050 1150 50  0001 C CNN
@@
 U 1 1 61037130
 P 6750 2600
-F 0 "R6" H 6820 2646 50  0000 L CNN
-F 1 "49R9" H 6820 2555 50  0000 L CNN
+F 0 "R6" H 6800 2650 50  0000 L CNN
+F 1 "49R9" H 6800 2550 50  0000 L CNN
 F 2 "Resistor_SMD:R_0603_1608Metric_Pad0.98x0.95mm_HandSolder" V 6680 2600 50  0001 C CNN
 F 3 "~" H 6750 2600 50  0001 C CNN
@@
 U 1 1 61046D5E
 P 7100 2850
-F 0 "R8" H 7030 2804 50  0000 R CNN
-F 1 "1k" H 7030 2895 50  0000 R CNN
+F 0 "R8" H 7050 2800 50  0000 R CNN
+F 1 "1k" H 7050 2900 50  0000 R CNN
 F 2 "Resistor_SMD:R_0603_1608Metric_Pad0.98x0.95mm_HandSolder" V 7030 2850 50  0001 C CNN
 F 3 "~" H 7100 2850 50  0001 C CNN
@@
 U 1 1 610445A2
 P 7300 2850
-F 0 "R9" H 7230 2804 50  0000 R CNN
-F 1 "1k" H 7230 2895 50  0000 R CNN
+F 0 "R9" H 7250 2800 50  0000 R CNN
+F 1 "1k" H 7250 2900 50  0000 R CNN
 F 2 "Resistor_SMD:R_0603_1608Metric_Pad0.98x0.95mm_HandSolder" V 7230 2850 50  0001 C CNN
 F 3 "~" H 7300 2850 50  0001 C CNN
@@
 U 1 1 6108521D
 P 7500 2550
-F 0 "C18" H 7615 2596 50  0000 L CNN
-F 1 "100n" H 7615 2505 50  0000 L CNN
+F 0 "C18" H 7500 2650 50  0000 L CNN
+F 1 "100n" H 7500 2450 50  0000 L CNN
 F 2 "Capacitor_SMD:C_0603_1608Metric_Pad1.05x0.95mm_HandSolder" H 7538 2400 50  0001 C CNN
 F 3 "~" H 7500 2550 50  0001 C CNN
@@
 U 1 1 61039AD2
 P 6750 1150
-F 0 "C17" H 6865 1196 50  0000 L CNN
-F 1 "100n" H 6865 1105 50  0000 L CNN
+F 0 "C17" H 6750 1250 50  0000 L CNN
+F 1 "100n" H 6750 1050 50  0000 L CNN
 F 2 "Capacitor_SMD:C_0603_1608Metric_Pad1.05x0.95mm_HandSolder" H 6788 1000 50  0001 C CNN
 F 3 "~" H 6750 1150 50  0001 C CNN
@@
 U 1 1 60F8EB2D
 P 6600 3000
-F 0 "C16" H 6715 3046 50  0000 L CNN
-F 1 "100n" H 6715 2955 50  0000 L CNN
+F 0 "C16" H 6600 3100 50  0000 L CNN
+F 1 "100n" H 6600 2900 50  0000 L CNN
 F 2 "Capacitor_SMD:C_0603_1608Metric_Pad1.05x0.95mm_HandSolder" H 6638 2850 50  0001 C CNN
 F 3 "~" H 6600 3000 50  0001 C CNN
@@
 U 1 1 610395CE
 P 6450 1150
-F 0 "R4" H 6520 1196 50  0000 L CNN
-F 1 "49R9" H 6520 1105 50  0000 L CNN
+F 0 "R4" H 6500 1200 50  0000 L CNN
+F 1 "49R9" H 6450 1000 50  0000 L CNN
 F 2 "Resistor_SMD:R_0603_1608Metric_Pad0.98x0.95mm_HandSolder" V 6380 1150 50  0001 C CNN
 F 3 "~" H 6450 1150 50  0001 C CNN
@@
 F 2 "Package_TO_SOT_SMD:SOT-223-3_TabPin2" H 2100 4950 50  0001 C CNN
 F 3 "http://www.ti.com/lit/ds/symlink/lm1117.pdf" H 2100 4950 50  0001 C CNN
+F 4 "Texas Instruments" H 2100 4950 50  0001 C CNN "Manufacturer"
+F 5 "LM1117IMPX-3.3/NOPB" H 2100 4950 50  0001 C CNN "Manufacturer PN"
 	1    2100 4950
 	1    0    0    -1
@@
 U 1 1 6113C12C
 P 4100 6900
-F 0 "C10" H 4215 6946 50  0000 L CNN
-F 1 "100n" H 4215 6855 50  0000 L CNN
+F 0 "C10" H 4100 7000 50  0000 L CNN
+F 1 "100n" H 4100 6800 50  0000 L CNN
 F 2 "Capacitor_SMD:C_0603_1608Metric_Pad1.05x0.95mm_HandSolder" H 4138 6750 50  0001 C CNN
 F 3 "~" H 4100 6900 50  0001 C CNN
@@
 U 1 1 611476FB
 P 3850 6900
-F 0 "C9" H 3965 6946 50  0000 L CNN
-F 1 "100n" H 3965 6855 50  0000 L CNN
+F 0 "C9" H 3850 7000 50  0000 L CNN
+F 1 "100n" H 3850 6800 50  0000 L CNN
 F 2 "Capacitor_SMD:C_0603_1608Metric_Pad1.05x0.95mm_HandSolder" H 3888 6750 50  0001 C CNN
 F 3 "~" H 3850 6900 50  0001 C CNN
@@
 U 1 1 61147A82
 P 4350 6900
-F 0 "C11" H 4465 6946 50  0000 L CNN
-F 1 "100n" H 4465 6855 50  0000 L CNN
+F 0 "C11" H 4350 7000 50  0000 L CNN
+F 1 "100n" H 4350 6800 50  0000 L CNN
 F 2 "Capacitor_SMD:C_0603_1608Metric_Pad1.05x0.95mm_HandSolder" H 4388 6750 50  0001 C CNN
 F 3 "~" H 4350 6900 50  0001 C CNN
@@
 U 1 1 61147D52
 P 4600 6900
-F 0 "C12" H 4715 6946 50  0000 L CNN
-F 1 "100n" H 4715 6855 50  0000 L CNN
+F 0 "C12" H 4600 7000 50  0000 L CNN
+F 1 "100n" H 4600 6800 50  0000 L CNN
 F 2 "Capacitor_SMD:C_0603_1608Metric_Pad1.05x0.95mm_HandSolder" H 4638 6750 50  0001 C CNN
 F 3 "~" H 4600 6900 50  0001 C CNN
@@
 U 1 1 61147FD8
 P 4850 6900
-F 0 "C13" H 4965 6946 50  0000 L CNN
-F 1 "100n" H 4965 6855 50  0000 L CNN
+F 0 "C13" H 4850 7000 50  0000 L CNN
+F 1 "100n" H 4850 6800 50  0000 L CNN
 F 2 "Capacitor_SMD:C_0603_1608Metric_Pad1.05x0.95mm_HandSolder" H 4888 6750 50  0001 C CNN
 F 3 "~" H 4850 6900 50  0001 C CNN
@@
 U 1 1 611484EB
 P 5100 6900
-F 0 "C14" H 5215 6946 50  0000 L CNN
-F 1 "100n" H 5215 6855 50  0000 L CNN
+F 0 "C14" H 5100 7000 50  0000 L CNN
+F 1 "100n" H 5100 6800 50  0000 L CNN
 F 2 "Capacitor_SMD:C_0603_1608Metric_Pad1.05x0.95mm_HandSolder" H 5138 6750 50  0001 C CNN
 F 3 "~" H 5100 6900 50  0001 C CNN
@@
 U 1 1 6114880A
 P 5350 6900
-F 0 "C15" H 5465 6946 50  0000 L CNN
-F 1 "100n" H 5465 6855 50  0000 L CNN
+F 0 "C15" H 5350 7000 50  0000 L CNN
+F 1 "100n" H 5350 6800 50  0000 L CNN
 F 2 "Capacitor_SMD:C_0603_1608Metric_Pad1.05x0.95mm_HandSolder" H 5388 6750 50  0001 C CNN
 F 3 "~" H 5350 6900 50  0001 C CNN
@@
 U 1 1 61188399
 P 1750 6900
-F 0 "C2" H 1865 6946 50  0000 L CNN
-F 1 "100n" H 1865 6855 50  0000 L CNN
+F 0 "C2" H 1750 7000 50  0000 L CNN
+F 1 "100n" H 1750 6800 50  0000 L CNN
 F 2 "Capacitor_SMD:C_0603_1608Metric_Pad1.05x0.95mm_HandSolder" H 1788 6750 50  0001 C CNN
 F 3 "~" H 1750 6900 50  0001 C CNN
@@
 U 1 1 611888D8
 P 2000 6900
-F 0 "C4" H 2115 6946 50  0000 L CNN
-F 1 "100n" H 2115 6855 50  0000 L CNN
+F 0 "C4" H 2000 7000 50  0000 L CNN
+F 1 "100n" H 2000 6800 50  0000 L CNN
 F 2 "Capacitor_SMD:C_0603_1608Metric_Pad1.05x0.95mm_HandSolder" H 2038 6750 50  0001 C CNN
 F 3 "~" H 2000 6900 50  0001 C CNN
@@
 U 1 1 61188E52
 P 2250 6900
-F 0 "C5" H 2365 6946 50  0000 L CNN
-F 1 "100n" H 2365 6855 50  0000 L CNN
+F 0 "C5" H 2250 7000 50  0000 L CNN
+F 1 "100n" H 2250 6800 50  0000 L CNN
 F 2 "Capacitor_SMD:C_0603_1608Metric_Pad1.05x0.95mm_HandSolder" H 2288 6750 50  0001 C CNN
 F 3 "~" H 2250 6900 50  0001 C CNN
@@
 U 1 1 61189171
 P 2500 6900
-F 0 "C7" H 2615 6946 50  0000 L CNN
-F 1 "100n" H 2615 6855 50  0000 L CNN
+F 0 "C7" H 2500 7000 50  0000 L CNN
+F 1 "100n" H 2500 6800 50  0000 L CNN
 F 2 "Capacitor_SMD:C_0603_1608Metric_Pad1.05x0.95mm_HandSolder" H 2538 6750 50  0001 C CNN
 F 3 "~" H 2500 6900 50  0001 C CNN
@@
 F 2 "Crystal:Crystal_HC18-U_Vertical" H 2100 1600 50  0001 C CNN
 F 3 "~" H 2100 1600 50  0001 C CNN
+F 4 "ECS" H 2100 1600 50  0001 C CNN "Manufacturer"
+F 5 "ECS-200-18-4X-CKM" H 2100 1600 50  0001 C CNN "Manufacturer PN"
 	1    2100 1600
 	-1   0    0    1
@@
 P 5700 4250
 F 0 "#PWR0122" H 5700 4000 50  0001 C CNN
-F 1 "GND" H 5705 4077 50  0000 C CNN
+F 1 "GND" H 5800 4250 50  0000 C CNN
 F 2 "" H 5700 4250 50  0001 C CNN
 F 3 "" H 5700 4250 50  0001 C CNN
